File: PCB/EDU-NXP/ON_BOARD_IO.sch (KiCad schematic (older format))
At the start: 64 parts, among them Q1 2N7000, Q10 2N7000, Q11 2N7000, Q12 2N7000, Q2 2N7000, Q3 2N7000, Q4 2N7000, Q5 2N7000, Q6 2N7000, Q7 2N7000, Q8 2N7000, Q9 2N7000, SW2 SW_PUSH, SW3 SW_PUSH, SW4 SW_PUSH, SW5 SW_PUSH

Commit message: Primera versión
Primera versión de la EDU - CIAA
Parts:
- removed R1, R2, R3, R4, R5, R6, R7: R, ~, symbol R
- removed S1: 7SEGM, ~, symbol 7SEGM
Other:
- moved on the sheet: LED0, LED1, LED2, LED3, Q1, Q10, Q11, Q12, Q2, Q3, Q4, Q5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

Commit message: Borrador del PCB
Parts:
- Q1, Q10, Q11, Q12, Q2, Q3, Q4, Q5, Q6, Q7, Q8, Q9: value 2N7000 -> 2N7002
- SW1: renamed from SW2; value SW_PUSH -> TEC_1
- SW2: renamed from SW3; value SW_PUSH -> TEC_2
- SW3: renamed from SW4; value SW_PUSH -> TEC_3
- SW4: renamed from SW5; value SW_PUSH -> TEC_4
- renumbered C4 to C10, C1 to C7, C2 to C8, C3 to C9, LED0 to LED1, LED1 to LED3, LED3 to LED4, R8 to R58, R9 to R59, R10 to R60, R11 to R61, R16 to R62, R17 to R63, R18 to R64, R19 to R65, R20 to R66, R21 to R67, R23 to R68, R24 to R69, R25 to R70, R26 to R71, R27 to R72, R28 to R73, R29 to R74, R30 to R75, R31 to R76, R41 to R77, R42 to R78, R43 to R79, R44 to R80, R45 to R81, R46 to R82, R47 to R83, R50 to R84, R51 to R85, R52 to R86, R53 to R87, R54 to R88, R55 to R89
