File: PCB/EDU-NXP/cpu.sch (KiCad schematic (older format))
At the start: 77 parts, among them J7 ZX62-AB-5PA, P8 Cortex-Debug, P9 FT_NC, SW1 SW_PUSH, U14 TXB0108, U16 LPC4337JBD144, U17 FT2232H, U19 93C46, X1 32.768K, X2 12MHz, X3 12MHz

Commit message: Versión con algunas mejoras
Connections:
- net labels removed: AUX_CLK, USB_AUX_DM, USB_AUX_DP
- wire segments 416 -> 415
