File: PCB/EDU-NXP/cpu.sch (KiCad schematic (older format))
At the start: 77 parts, among them J7 ZX62-AB-5PA, P8 Cortex-Debug, P9 FT_NC, SW1 SW_PUSH, U14 TXB0108, U16 LPC4337JBD144, U17 FT2232H, U19 93C46, X1 32.768K, X2 12MHz, X3 12MHz

Commit message: Primera versión
Primera versión de la EDU - CIAA
Connections:
- net labels removed: 7SEG_a, 7SEG_b, 7SEG_c, 7SEG_d, 7SEG_e, 7SEG_f, 7SEG_g, EMC_CLK0, SPIFI_CS, SPIFI_IO2, SPIFI_IO3, SPIFI_MISO, SPIFI_MOSI, SPIFI_SCK
- wire segments 415 -> 416
- no-connect marks 4 -> 41

Commit message: Borrador del PCB
Parts:
- R103: renamed from R97; value 12K -> 12K 1%
- SW5: renamed from SW1; value SW_PUSH -> RESET
- renumbered C79 to C11, C81 to C12, C82 to C13, C83 to C14, C84 to C15, C85 to C16, C69 to C17, C86 to C18, C87 to C19, C47 to C20, C48 to C21, C49 to C22, C50 to C23, C51 to C24, C52 to C25, C53 to C26, C54 to C27, C55 to C28, C56 to C29, C57 to C30, C58 to C31, C59 to C32, C60 to C33, C90 to C34, C80 to C35, C77 to C36, C78 to C37, C67 to C38, C68 to C39, C61 to C40, C70 to C41, C71 to C42, C72 to C43, C73 to C44, C74 to C45, C75 to C46, C76 to C47, C62 to C48, FB7 to FB5, FB11 to FB6, FB9 to FB7, J7 to J3, JP15 to JP5, P8 to P3, P9 to P4, R102 to R100, R104 to R101, R103 to R102, R98 to R104, R84 to R105, R85 to R106, R86 to R107, R87 to R108, R88 to R109, R89 to R110, R96 to R91, R95 to R92, R91 to R93, R92 to R94, R99 to R95, R93 to R96, R100 to R97, R94 to R98, R101 to R99, TR1 to TR2, U16 to U4, U19 to U5, U17 to U6, U14 to U7
Connections:
- net GND: now also C39.2; no longer C39.1
- net USB_JTAG_DM: now also TR2.3; no longer TR2.2
- net USB_JTAG_DP: now also TR2.2; no longer TR2.3
- net XTAL1: now also C14.2, R91.1, X2.1; no longer C13.2, R91.2, X2.2
- net XTAL2: now also C13.2, R91.2, X2.2; no longer C14.2, R91.1, X2.1
- net at C38.1, FB8.1, U6.9 (VPLL): now also C39.1; no longer C39.2
- net at TR2.1: now also J3.3 (P3); no longer J3.2 (P2)
- net at TR2.4: now also J3.2 (P2); no longer J3.3 (P3)
- net USB_PPWR: no longer names the net of U4.79 (P6_3)
- net USB_PWR_FAULT: no longer names the net of U4.83 (P6_6)
- no-connect marks 41 -> 43
