File: PCB/EDU-NXP/edu-ciaa-nxp.sch (KiCad schematic (older format))
At the start: 15 parts

Commit message: Versión con algunas mejoras
Connections:
- wire segments 89 -> 87
Changed lines of the file:
@@
 Sheet 1 7
 Title "CIAA NXP"
-Date "10 jun 2014"
+Date "12 jun 2014"
 Rev "1.0"
 Comp ""
@@
 Wire Wire Line
 	4800 2600 3600 2600
-Wire Wire Line
-	4800 3750 3600 3750
-Wire Wire Line
-	3600 3650 4800 3650
 $Comp
 L GS2 GS4
@@
 Wire Wire Line
 	4250 6500 3600 6500
-Wire Wire Line
-	3600 6600 4800 6600
 $Comp
 L CONN_1 H1
@@
 F22 "USB_VBUS" I R 7050 4150 60
 F23 "USB_ID" I R 7050 4250 60
-F24 "USB_AUX_DP" B L 4800 3650 60
-F25 "USB_AUX_DM" B L 4800 3750 60
-F26 "I2C_SCL" O R 7050 1750 60
-F27 "I2C_SDA" B R 7050 1650 60
-F28 "ENET_MDC" O R 7050 2800 60
-F29 "RS485_TXD" O R 7050 3400 60
-F30 "RS485_RXD" I R 7050 3500 60
-F31 "RESET" O L 4800 6850 60
-F32 "SPIFI_CS" O R 7050 1050 60
-F33 "SPIFI_SCK" O R 7050 1150 60
-F34 "SPIFI_MOSI" B R 7050 1250 60
-F35 "SPIFI_MISO" B R 7050 1350 60
-F36 "SPIFI_IO2" B R 7050 1450 60
-F37 "SPIFI_IO3" B R 7050 1550 60
-F38 "USB_PPWR" O R 7050 4350 60
-F39 "USB_PWR_FAULT" O R 7050 4450 60
-F40 "USB_DEBUG_VBUS" O L 4800 6600 60
-F41 "PULS_0" I R 7050 5650 60
-F42 "PULS_1" I R 7050 5750 60
-F43 "PULS_2" I R 7050 5850 60
-F44 "PULS_3" I R 7050 5950 60
-F45 "TEC_COL0" O L 4800 3950 60
-F46 "7SEG_a" I R 7050 4800 60
-F47 "7SEG_b" I R 7050 4900 60
-F48 "7SEG_c" I R 7050 5000 60
-F49 "7SEG_d" I R 7050 5100 60
-F50 "7SEG_e" I R 7050 5200 60
-F51 "7SEG_f" I R 7050 5300 60
-F52 "7SEG_g" I R 7050 5400 60
-F53 "TEC_F0" O L 4800 4250 60
-F54 "ADC0_1" I L 4800 5950 60
-F55 "TEC_F1" O L 4800 4350 60
-F56 "DAC" O L 4800 5850 60
-F57 "TEC_F3" O L 4800 4550 60
-F58 "TEC_F2" O L 4800 4450 60
-F59 "LCD1" O L 4800 5250 60
-F60 "LCD2" O L 4800 5350 60
-F61 "LCD3" O L 4800 5450 60
-F62 "LCD_RS" O L 4800 5650 60
-F63 "LCD__EN" O L 4800 5750 60
-F64 "LCD4" O L 4800 5550 60
-F65 "LED2_R" O R 7050 6300 60
-F66 "LED2_G" O R 7050 6400 60
-F67 "LED2_B" O R 7050 6500 60
-F68 "LED3_R" O R 7050 6650 60
-F69 "LED3_G" O R 7050 6750 60
-F70 "LED3_B" O R 7050 6850 60
-F71 "GPIO4" B L 4800 1450 60
-F72 "CAN_RD" I L 4800 5100 60
-F73 "CAN_TD" O L 4800 5000 60
-F74 "GPIO5" B L 4800 1550 60
-F75 "WAKEUP0" I L 4800 2150 60
-F76 "TEC_COL1" O L 4800 4050 60
-F77 "TEC_COL2" O L 4800 4150 60
-F78 "GPIO6" B L 4800 1650 60
-F79 "ADC0_3" I L 4800 4800 60
-F80 "ISP" I R 7050 1900 60
-F81 "ADC0_2" I L 4800 4900 60
-F82 "GPIO8" B L 4800 1850 60
-F83 "GPIO7" B L 4800 1750 60
+F24 "I2C_SCL" O R 7050 1750 60
+F25 "I2C_SDA" B R 7050 1650 60
+F26 "ENET_MDC" O R 7050 2800 60
+F27 "RS485_TXD" O R 7050 3400 60
+F28 "RS485_RXD" I R 7050 3500 60
+F29 "RESET" O L 4800 6850 60
+F30 "SPIFI_CS" O R 7050 1050 60
+F31 "SPIFI_SCK" O R 7050 1150 60
+F32 "SPIFI_MOSI" B R 7050 1250 60
+F33 "SPIFI_MISO" B R 7050 1350 60
+F34 "SPIFI_IO2" B R 7050 1450 60
+F35 "SPIFI_IO3" B R 7050 1550 60
+F36 "USB_PPWR" O R 7050 4350 60
+F37 "USB_PWR_FAULT" O R 7050 4450 60
+F38 "PULS_0" I R 7050 5650 60
+F39 "PULS_1" I R 7050 5750 60
+F40 "PULS_2" I R 7050 5850 60
+F41 "PULS_3" I R 7050 5950 60
+F42 "TEC_COL0" O L 4800 3950 60
+F43 "7SEG_a" I R 7050 4800 60
+F44 "7SEG_b" I R 7050 4900 60
+F45 "7SEG_c" I R 7050 5000 60
+F46 "7SEG_d" I R 7050 5100 60
+F47 "7SEG_e" I R 7050 5200 60
+F48 "7SEG_f" I R 7050 5300 60
+F49 "7SEG_g" I R 7050 5400 60
+F50 "TEC_F0" O L 4800 4250 60
+F51 "ADC0_1" I L 4800 5950 60
+F52 "TEC_F1" O L 4800 4350 60
+F53 "DAC" O L 4800 5850 60
+F54 "TEC_F3" O L 4800 4550 60
+F55 "TEC_F2" O L 4800 4450 60
+F56 "LCD1" O L 4800 5250 60
+F57 "LCD2" O L 4800 5350 60
+F58 "LCD3" O L 4800 5450 60
+F59 "LCD_RS" O L 4800 5650 60
+F60 "LCD__EN" O L 4800 5750 60
+F61 "LCD4" O L 4800 5550 60
+F62 "LED2_R" O R 7050 6300 60
+F63 "LED2_G" O R 7050 6400 60
+F64 "LED2_B" O R 7050 6500 60
+F65 "LED3_R" O R 7050 6650 60
+F66 "LED3_G" O R 7050 6750 60
+F67 "LED3_B" O R 7050 6850 60
+F68 "GPIO4" B L 4800 1450 60
+F69 "CAN_RD" I L 4800 5100 60
+F70 "CAN_TD" O L 4800 5000 60
+F71 "GPIO5" B L 4800 1550 60
+F72 "WAKEUP0" I L 4800 2150 60
+F73 "TEC_COL1" O L 4800 4050 60
+F74 "TEC_COL2" O L 4800 4150 60
+F75 "GPIO6" B L 4800 1650 60
+F76 "ADC0_3" I L 4800 4800 60
+F77 "ISP" I R 7050 1900 60
+F78 "ADC0_2" I L 4800 4900 60
+F79 "GPIO8" B L 4800 1850 60
+F80 "GPIO7" B L 4800 1750 60
+F81 "USB_DEBUG_VBUS" O L 4800 6600 60
 $EndSheet
 Wire Wire Line
@@
 F10 "I2C_SDA" B R 3600 2950 60
 F11 "I2C_SCL" I R 3600 3050 60
-F12 "USB_DP" B R 3600 3650 60
-F13 "USB_DM" B R 3600 3750 60
-F14 "SPI_MISO" O R 3600 2700 60
-F15 "SPI_MOSI" I R 3600 2800 60
-F16 "SPI_SCK" I R 3600 2600 60
-F17 "GPIO6" B R 3600 1650 60
-F18 "ENET_RXD1" I L 2400 3400 60
-F19 "ENET_TX_EN" I L 2400 3500 60
-F20 "TEC_COL0" I R 3600 3950 60
-F21 "ENET_RXD0" I L 2400 3600 60
-F22 "ENET_CRS_DV" I L 2400 3700 60
-F23 "ENET_MDIO" B L 2400 3800 60
-F24 "ENET_TXD0" O L 2400 3900 60
-F25 "ENET_REF_CLK" I L 2400 4100 60
-F26 "ENET_TXD1" O L 2400 4000 60
-F27 "TEC_F0" O R 3600 4250 60
-F28 "ADC0_1" I R 3600 5950 60
-F29 "TEC_F1" O R 3600 4350 60
-F30 "DAC" O R 3600 5850 60
-F31 "TEC_F2" O R 3600 4450 60
-F32 "TEC_F3" O R 3600 4550 60
-F33 "LCD1" O R 3600 5250 60
-F34 "LCD2" O R 3600 5350 60
-F35 "LCD3" O R 3600 5450 60
-F36 "LCD_RS" O R 3600 5650 60
-F37 "LCD_EN" O R 3600 5750 60
-F38 "LCD4" O R 3600 5550 60
-F39 "CAN_RD" I R 3600 5100 60
-F40 "CAN_TD" O R 3600 5000 60
-F41 "WAKEUP" I R 3600 2150 60
-F42 "TEC_COL1" I R 3600 4050 60
-F43 "TEC_COL2" I R 3600 4150 60
-F44 "ISP" I L 2400 1250 60
-F45 "ADC0_3" I R 3600 4800 60
-F46 "ADC0_2" I R 3600 4900 60
+F12 "SPI_MISO" O R 3600 2700 60
+F13 "SPI_MOSI" I R 3600 2800 60
+F14 "SPI_SCK" I R 3600 2600 60
+F15 "GPIO6" B R 3600 1650 60
+F16 "ENET_RXD1" I L 2400 3400 60
+F17 "ENET_TX_EN" I L 2400 3500 60
+F18 "TEC_COL0" I R 3600 3950 60
+F19 "ENET_RXD0" I L 2400 3600 60
+F20 "ENET_CRS_DV" I L 2400 3700 60
+F21 "ENET_MDIO" B L 2400 3800 60
+F22 "ENET_TXD0" O L 2400 3900 60
+F23 "ENET_REF_CLK" I L 2400 4100 60
+F24 "ENET_TXD1" O L 2400 4000 60
+F25 "TEC_F0" O R 3600 4250 60
+F26 "ADC0_1" I R 3600 5950 60
+F27 "TEC_F1" O R 3600 4350 60
+F28 "DAC" O R 3600 5850 60
+F29 "TEC_F2" O R 3600 4450 60
+F30 "TEC_F3" O R 3600 4550 60
+F31 "LCD1" O R 3600 5250 60
+F32 "LCD2" O R 3600 5350 60
+F33 "LCD3" O R 3600 5450 60
+F34 "LCD_RS" O R 3600 5650 60
+F35 "LCD_EN" O R 3600 5750 60
+F36 "LCD4" O R 3600 5550 60
+F37 "CAN_RD" I R 3600 5100 60
+F38 "CAN_TD" O R 3600 5000 60
+F39 "WAKEUP" I R 3600 2150 60
+F40 "TEC_COL1" I R 3600 4050 60
+F41 "TEC_COL2" I R 3600 4150 60
+F42 "ISP" I L 2400 1250 60
+F43 "ADC0_3" I R 3600 4800 60
+F44 "ADC0_2" I R 3600 4900 60
 $EndSheet
 Wire Wire Line
@@
 F1 "fuente.sch" 50
 F2 "USB_VBUS" I R 3600 6400 60
-F3 "USB_VBUS3" I R 3600 6600 60
-F4 "USB_VBUS2" I R 3600 6500 60
+F3 "USB_VBUS2" I R 3600 6500 60
+F4 "USB_VBUS3" I R 3600 6600 60
 $EndSheet
+Wire Wire Line
+	4800 6600 3600 6600
 $EndSCHEMATC
