File: PCB/EDU-NXP/edu-ciaa-nxp.sch (KiCad schematic (older format))
At the start: 15 parts

Commit message: Primera versión
Primera versión de la EDU - CIAA
Connections:
- net labels removed: GPIO7, GPIO8
- wire segments 95 -> 88
- no-connect marks 1 -> 14
Other:
- note added: "Índice:\n1. Esquemático jerárquico\n2. RS485\n3. USB OTG\n4. GPIO\n5. Fuente de alimentación\n6. On Board IO\n7. CPU\n"
- note removed: "Índice:\n1. Esquemático jerárquico\n2. CPU\n3. RS485/RS232\n4. USB OTG\n5. GPIO\n6. Fuente de alimentación"
Changed lines of the file:
@@
 encoding utf-8
 Sheet 1 7
-Title "CIAA NXP"
-Date "13 jun 2014"
+Title "EDU CIAA NXP"
+Date "14 jun 2014"
 Rev "1.0"
 Comp ""
@@
 S 8300 2550 1150 600
 U 52C1F703
-F0 "RS485_RS232_CAN" 50
+F0 "RS485" 50
 F1 "rsS485_rs232_can.sch" 50
 F2 "RS485_RXD" O L 8300 3050 60
@@
 Text Label 4450 6850 0    60   ~ 0
 RESET
-Text Label 7450 3700 0    60   ~ 0
-USB_VBUS
 Text Label 4250 6400 2    60   ~ 0
 USB_VBUS
@@
 Wire Wire Line
 	7050 4000 7800 4000
-Text Notes 8650 1350 0    118  ~ 0
-Índice:\n1. Esquemático jerárquico\n2. CPU\n3. RS485/RS232\n4. USB OTG\n5. GPIO\n6. Fuente de alimentación
+Text Notes 8350 850  0    118  ~ 0
+Índice:\n1. Esquemático jerárquico\n2. RS485\n3. USB OTG\n4. GPIO\n5. Fuente de alimentación\n6. On Board IO\n7. CPU\n
 Wire Wire Line
 	3600 2150 4800 2150
 NoConn ~ 3600 2350
-Text Label 7300 3900 0    60   ~ 0
-GPIO7
-Text Label 7300 4000 0    60   ~ 0
-GPIO8
 Wire Wire Line
 	3600 1750 4800 1750
@@
 Text Label 1750 3500 0    60   ~ 0
 ENET_TX_EN
-$Sheet
-S 4800 950  2250 6300
-U 52C1CAF4
-F0 "CPU" 50
-F1 "cpu.sch" 50
-F2 "ENET_RXD1" I R 7050 1900 60
-F3 "ENET_TX_EN" O R 7050 2700 60
-F4 "GPIO0" B L 4800 1050 60
-F5 "GPIO1" B L 4800 1150 60
-F6 "ENET_RXD0" I R 7050 2000 60
-F7 "ENET_CRS_DV" I R 7050 2100 60
-F8 "ENET_MDIO" B R 7050 2200 60
-F9 "ENET_TXD0" O R 7050 2300 60
-F10 "ENET_REF_CLK" I R 7050 2500 60
-F11 "ENET_TXD1" O R 7050 2400 60
-F12 "GPIO2" B L 4800 1250 60
-F13 "GPIO3" B L 4800 1350 60
-F14 "SPI_SCK" O L 4800 2600 60
-F15 "RS232_TXD" O L 4800 2300 60
-F16 "RS232_RXD" I L 4800 2400 60
-F17 "SPI_MISO" I L 4800 2700 60
-F18 "SPI_MOSI" O L 4800 2800 60
-F19 "RS485_DIR" O R 7050 2850 60
-F20 "USB_DP" B R 7050 3500 60
-F21 "USB_DM" B R 7050 3600 60
-F22 "USB_VBUS" I R 7050 3700 60
-F23 "USB_ID" I R 7050 3800 60
-F24 "ENET_MDC" O R 7050 2600 60
-F25 "RS485_TXD" O R 7050 2950 60
-F26 "RS485_RXD" I R 7050 3050 60
-F27 "RESET" O L 4800 6850 60
-F28 "SPIFI_CS" O R 7050 1050 60
-F29 "SPIFI_SCK" O R 7050 1150 60
-F30 "SPIFI_MOSI" B R 7050 1250 60
-F31 "SPIFI_MISO" B R 7050 1350 60
-F32 "SPIFI_IO2" B R 7050 1450 60
-F33 "SPIFI_IO3" B R 7050 1550 60
-F34 "USB_PPWR" O R 7050 3900 60
-F35 "USB_PWR_FAULT" O R 7050 4000 60
-F36 "PULS_0" I R 7050 5200 60
-F37 "PULS_1" I R 7050 5300 60
-F38 "PULS_2" I R 7050 5400 60
-F39 "PULS_3" I R 7050 5500 60
-F40 "TEC_COL0" O L 4800 3950 60
-F41 "7SEG_a" I R 7050 4350 60
-F42 "7SEG_b" I R 7050 4450 60
-F43 "7SEG_c" I R 7050 4550 60
-F44 "7SEG_d" I R 7050 4650 60
-F45 "7SEG_e" I R 7050 4750 60
-F46 "7SEG_f" I R 7050 4850 60
-F47 "7SEG_g" I R 7050 4950 60
-F48 "TEC_F0" O L 4800 4250 60
-F49 "ADC0_1" I L 4800 5950 60
-F50 "TEC_F1" O L 4800 4350 60
-F51 "DAC" O L 4800 5850 60
-F52 "TEC_F3" O L 4800 4550 60
-F53 "TEC_F2" O L 4800 4450 60
-F54 "LCD1" O L 4800 5250 60
-F55 "LCD2" O L 4800 5350 60
-F56 "LCD3" O L 4800 5450 60
-F57 "LCD_RS" O L 4800 5650 60
-F58 "LCD__EN" O L 4800 5750 60
-F59 "LCD4" O L 4800 5550 60
-F60 "LED2_R" O R 7050 6450 60
-F61 "LED2_G" O R 7050 6550 60
-F62 "LED2_B" O R 7050 6650 60
-F63 "LED3_R" O R 7050 6800 60
-F64 "LED3_G" O R 7050 6900 60
-F65 "LED3_B" O R 7050 7000 60
-F66 "GPIO4" B L 4800 1450 60
-F67 "CAN_RD" I L 4800 5100 60
-F68 "CAN_TD" O L 4800 5000 60
-F69 "GPIO5" B L 4800 1550 60
-F70 "WAKEUP0" I L 4800 2150 60
-F71 "TEC_COL1" O L 4800 4050 60
-F72 "TEC_COL2" O L 4800 4150 60
-F73 "GPIO6" B L 4800 1650 60
-F74 "ADC0_3" I L 4800 4800 60
-F75 "ISP" I R 7050 1700 60
-F76 "ADC0_2" I L 4800 4900 60
-F77 "GPIO8" B L 4800 1850 60
-F78 "GPIO7" B L 4800 1750 60
-F79 "USB_DEBUG_VBUS" O L 4800 6600 60
-F80 "I2C_SCL" O L 4800 3050 60
-F81 "I2C_SDA" B L 4800 2950 60
-F82 "LED1_R" O R 7050 6100 60
-F83 "LED1_G" O R 7050 6200 60
-F84 "LED1_B" O R 7050 6300 60
-F85 "LED0_R" O R 7050 5750 60
-F86 "LED0_G" O R 7050 5850 60
-F87 "LED0_B" O R 7050 5950 60
-$EndSheet
 Wire Wire Line
 	7050 5500 8300 5500
@@
 Wire Wire Line
 	3600 3950 4800 3950
-Wire Wire Line
-	7050 4950 8300 4950
-Wire Wire Line
-	7050 4350 8300 4350
-Wire Wire Line
-	8300 4450 7050 4450
-Wire Wire Line
-	7050 4550 8300 4550
-Wire Wire Line
-	8300 4650 7050 4650
-Wire Wire Line
-	7050 4750 8300 4750
-Wire Wire Line
-	8300 4850 7050 4850
 Text Label 7100 2000 0    60   ~ 0
 ENET_RXD0
@@
 ENET_MDC
 Wire Wire Line
-	1750 4300 2400 4300
-Wire Wire Line
 	2400 4000 1750 4000
 Wire Wire Line
@@
 Wire Wire Line
 	2400 4200 1750 4200
-Text Label 1750 4300 0    60   ~ 0
-ENET_TX_EN
 Text Label 1750 4000 0    60   ~ 0
 ENET_TXD1
@@
 F45 "RS232_TXD" O R 3600 2300 60
 F46 "RS232_RXD" I R 3600 2400 60
+F47 "ENET_MDC" O L 2400 4200 60
+F48 "RESET" O L 2400 5850 60
 $EndSheet
 Wire Wire Line
@@
 F4 "PULS_2" I L 8300 5400 60
 F5 "PULS_3" I L 8300 5500 60
-F6 "7SEGM_a" O L 8300 4350 60
-F7 "7SEGM_b" O L 8300 4450 60
-F8 "7SEGM_c" O L 8300 4550 60
-F9 "7SEGM_d" O L 8300 4650 60
-F10 "7SEGM_e" O L 8300 4750 60
-F11 "7SEGM_f" O L 8300 4850 60
-F12 "7SEGM_g" O L 8300 4950 60
-F13 "LED2_R" O L 8300 6450 60
-F14 "LED2_G" O L 8300 6550 60
-F15 "LED2_B" O L 8300 6650 60
-F16 "LED3_R" O L 8300 6800 60
-F17 "LED3_G" O L 8300 6900 60
-F18 "LED3_B" O L 8300 7000 60
-F19 "LED0_B" O L 8300 5950 60
-F20 "LED0_G" O L 8300 5850 60
-F21 "LED0_R" O L 8300 5750 60
-F22 "LED1_B" O L 8300 6300 60
-F23 "LED1_G" O L 8300 6200 60
-F24 "LED1_R" O L 8300 6100 60
+F6 "LED2_R" O L 8300 6450 60
+F7 "LED2_G" O L 8300 6550 60
+F8 "LED2_B" O L 8300 6650 60
+F9 "LED3_R" O L 8300 6800 60
+F10 "LED3_G" O L 8300 6900 60
+F11 "LED3_B" O L 8300 7000 60
+F12 "LED0_B" O L 8300 5950 60
+F13 "LED0_G" O L 8300 5850 60
+F14 "LED0_R" O L 8300 5750 60
+F15 "LED1_B" O L 8300 6300 60
+F16 "LED1_G" O L 8300 6200 60
+F17 "LED1_R" O L 8300 6100 60
 $EndSheet
 Wire Wire Line
@@
 Wire Wire Line
 	7050 6300 8300 6300
+NoConn ~ 9750 3900
+NoConn ~ 9750 4000
+NoConn ~ 9750 4100
+NoConn ~ 10300 3900
+NoConn ~ 10300 4000
+NoConn ~ 10300 4100
+NoConn ~ 10300 4550
+NoConn ~ 10300 4700
+NoConn ~ 10300 4850
+NoConn ~ 10300 5000
+NoConn ~ 10300 5200
+NoConn ~ 10300 5300
+NoConn ~ 10300 5400
+$Sheet
+S 4800 950  2250 6300
+U 52C1CAF4
+F0 "CPU" 50
+F1 "cpu.sch" 50
+F2 "ENET_RXD1" I R 7050 1900 60
+F3 "ENET_TX_EN" O R 7050 2700 60
+F4 "GPIO0" B L 4800 1050 60
+F5 "GPIO1" B L 4800 1150 60
+F6 "ENET_RXD0" I R 7050 2000 60
+F7 "ENET_CRS_DV" I R 7050 2100 60
+F8 "ENET_MDIO" B R 7050 2200 60
+F9 "ENET_TXD0" O R 7050 2300 60
+F10 "ENET_REF_CLK" I R 7050 2500 60
+F11 "ENET_TXD1" O R 7050 2400 60
+F12 "GPIO2" B L 4800 1250 60
+F13 "GPIO3" B L 4800 1350 60
+F14 "SPI_SCK" O L 4800 2600 60
+F15 "RS232_TXD" O L 4800 2300 60
+F16 "RS232_RXD" I L 4800 2400 60
+F17 "SPI_MISO" I L 4800 2700 60
+F18 "SPI_MOSI" O L 4800 2800 60
+F19 "RS485_DIR" O R 7050 2850 60
+F20 "USB_DP" B R 7050 3500 60
+F21 "USB_DM" B R 7050 3600 60
+F22 "USB_VBUS" I R 7050 3700 60
+F23 "USB_ID" I R 7050 3800 60
+F24 "ENET_MDC" O R 7050 2600 60
+F25 "RS485_TXD" O R 7050 2950 60
+F26 "RS485_RXD" I R 7050 3050 60
+F27 "RESET" O L 4800 6850 60
+F28 "USB_PPWR" O R 7050 3900 60
+F29 "USB_PWR_FAULT" O R 7050 4000 60
+F30 "PULS_0" I R 7050 5200 60
+F31 "PULS_1" I R 7050 5300 60
+F32 "PULS_2" I R 7050 5400 60
+F33 "PULS_3" I R 7050 5500 60
+F34 "TEC_COL0" O L 4800 3950 60
+F35 "TEC_F0" O L 4800 4250 60
+F36 "ADC0_1" I L 4800 5950 60
+F37 "TEC_F1" O L 4800 4350 60
+F38 "DAC" O L 4800 5850 60
+F39 "TEC_F3" O L 4800 4550 60
+F40 "TEC_F2" O L 4800 4450 60
+F41 "LCD1" O L 4800 5250 60
+F42 "LCD2" O L 4800 5350 60
+F43 "LCD3" O L 4800 5450 60
+F44 "LCD_RS" O L 4800 5650 60
+F45 "LCD__EN" O L 4800 5750 60
+F46 "LCD4" O L 4800 5550 60
+F47 "LED2_R" O R 7050 6450 60
+F48 "LED2_G" O R 7050 6550 60
+F49 "LED2_B" O R 7050 6650 60
+F50 "LED3_R" O R 7050 6800 60
+F51 "LED3_G" O R 7050 6900 60
+F52 "LED3_B" O R 7050 7000 60
+F53 "GPIO4" B L 4800 1450 60
+F54 "CAN_RD" I L 4800 5100 60
+F55 "CAN_TD" O L 4800 5000 60
+F56 "GPIO5" B L 4800 1550 60
+F57 "WAKEUP0" I L 4800 2150 60
+F58 "TEC_COL1" O L 4800 4050 60
+F59 "TEC_COL2" O L 4800 4150 60
+F60 "GPIO6" B L 4800 1650 60
+F61 "ADC0_3" I L 4800 4800 60
+F62 "ISP" I R 7050 1700 60
+F63 "ADC0_2" I L 4800 4900 60
+F64 "GPIO8" B L 4800 1850 60
+F65 "GPIO7" B L 4800 1750 60
+F66 "USB_DEBUG_VBUS" O L 4800 6600 60
+F67 "I2C_SCL" O L 4800 3050 60
+F68 "I2C_SDA" B L 4800 2950 60
+F69 "LED1_R" O R 7050 6100 60
+F70 "LED1_G" O R 7050 6200 60
+F71 "LED1_B" O R 7050 6300 60
+F72 "LED0_R" O R 7050 5750 60
+F73 "LED0_G" O R 7050 5850 60
+F74 "LED0_B" O R 7050 5950 60
+$EndSheet
+Wire Wire Line
+	2400 5850 2050 5850
+Text Label 2050 5850 0    60   ~ 0
+RESET
+Text Label 7450 3700 0    60   ~ 0
+USB_VBUS
 $EndSCHEMATC

Commit message: Borrador del PCB
Parts:
- removed GS4, GS5: GS2, symbol GS2
- removed H5, H6, H7: 4mm, symbol CONN_1
Connections:
- net labels removed: VBUS_GPIO
- wire segments 88 -> 83
- no-connect marks 14 -> 10
Changed lines of the file:
@@
 Sheet 1 7
 Title "EDU CIAA NXP"
-Date "14 jun 2014"
+Date "2 jul 2014"
 Rev "1.0"
 Comp ""
@@
 F0 "USB OTG" 50
 F1 "usb_otg.sch" 50
-F2 "USB0_PPWR" I L 8300 3900 60
-F3 "USB0_PWR_FAULT" I L 8300 4000 60
-F4 "USB_VBUS" O L 8300 3700 60
-F5 "USB_DM" B L 8300 3600 60
-F6 "USB_DP" B L 8300 3500 60
-F7 "USB_ID" O L 8300 3800 60
+F2 "USB_VBUS" O L 8300 3700 60
+F3 "USB_DM" B L 8300 3600 60
+F4 "USB_DP" B L 8300 3500 60
+F5 "USB_ID" O L 8300 3800 60
 $EndSheet
 Wire Wire Line
@@
 Wire Wire Line
 	8300 2850 7050 2850
-Wire Wire Line
-	7050 2950 8300 2950
 Wire Wire Line
 	8300 3050 7050 3050
@@
 Wire Wire Line
 	4800 2600 3600 2600
-$Comp
-L GS2 GS4
-U 1 1 52CC05DA
-P 8000 3900
-F 0 "GS4" V 7950 3700 50  0000 C CNN
-F 1 "GS2" V 8100 3751 40  0001 C CNN
-F 2 "" H 8000 3900 60  0000 C CNN
-F 3 "" H 8000 3900 60  0000 C CNN
-	1    8000 3900
-	0    -1   -1   0
-$EndComp
-$Comp
-L GS2 GS5
-U 1 1 52CC09B8
-P 8000 4000
-F 0 "GS5" V 7950 3800 50  0000 C CNN
-F 1 "GS2" V 8100 3851 40  0001 C CNN
-F 2 "" H 8000 4000 60  0000 C CNN
-F 3 "" H 8000 4000 60  0000 C CNN
-	1    8000 4000
-	0    -1   -1   0
-$EndComp
-Wire Wire Line
-	8200 3900 8300 3900
-Wire Wire Line
-	8300 4000 8200 4000
-Wire Wire Line
-	7050 3900 7800 3900
-Wire Wire Line
-	7050 4000 7800 4000
 Text Notes 8350 850  0    118  ~ 0
 Índice:\n1. Esquemático jerárquico\n2. RS485\n3. USB OTG\n4. GPIO\n5. Fuente de alimentación\n6. On Board IO\n7. CPU\n
 Wire Wire Line
 	3600 2150 4800 2150
-NoConn ~ 3600 2350
 Wire Wire Line
 	3600 1750 4800 1750
 Wire Wire Line
 	3600 1850 4800 1850
-Text Label 4250 6500 2    60   ~ 0
-VBUS_GPIO
-Wire Wire Line
-	4250 6500 3600 6500
 $Comp
 L CONN_1 H1
@@
 Text Notes 9750 3600 0    60   ~ 0
 fiduciales\n\nTOP       BOTTOM
-$Comp
-L CONN_1 H5
-U 1 1 534892C5
-P 10450 5200
-F 0 "H5" H 10530 5200 40  0000 L CNN
-F 1 "4mm" H 10450 5255 157 0001 C CNN
-F 2 "" H 10450 5200 60  0000 C CNN
-F 3 "" H 10450 5200 60  0000 C CNN
-	1    10450 5200
-	1    0    0    -1
-$EndComp
-$Comp
-L CONN_1 H6
-U 1 1 534892CB
-P 10450 5300
-F 0 "H6" H 10530 5300 40  0000 L CNN
-F 1 "4mm" H 10450 5355 157 0001 C CNN
-F 2 "" H 10450 5300 60  0000 C CNN
-F 3 "" H 10450 5300 60  0000 C CNN
-	1    10450 5300
-	1    0    0    -1
-$EndComp
-$Comp
-L CONN_1 H7
-U 1 1 534892D1
-P 10450 5400
-F 0 "H7" H 10530 5400 40  0000 L CNN
-F 1 "4mm" H 10450 5455 157 0001 C CNN
-F 2 "" H 10450 5400 60  0000 C CNN
-F 3 "" H 10450 5400 60  0000 C CNN
-	1    10450 5400
-	1    0    0    -1
-$EndComp
 Wire Wire Line
 	1750 3400 2400 3400
@@
 F1 "fuente.sch" 50
 F2 "USB_VBUS" I R 3600 6400 60
-F3 "USB_VBUS2" I R 3600 6500 60
-F4 "USB_VBUS3" I R 3600 6600 60
+F3 "USB_VBUS2" I R 3600 6600 60
 $EndSheet
 Wire Wire Line
@@
 NoConn ~ 10300 4850
 NoConn ~ 10300 5000
-NoConn ~ 10300 5200
-NoConn ~ 10300 5300
-NoConn ~ 10300 5400
 $Sheet
 S 4800 950  2250 6300
@@
 F23 "USB_ID" I R 7050 3800 60
 F24 "ENET_MDC" O R 7050 2600 60
-F25 "RS485_TXD" O R 7050 2950 60
-F26 "RS485_RXD" I R 7050 3050 60
-F27 "RESET" O L 4800 6850 60
-F28 "USB_PPWR" O R 7050 3900 60
-F29 "USB_PWR_FAULT" O R 7050 4000 60
-F30 "PULS_0" I R 7050 5200 60
-F31 "PULS_1" I R 7050 5300 60
-F32 "PULS_2" I R 7050 5400 60
-F33 "PULS_3" I R 7050 5500 60
-F34 "TEC_COL0" O L 4800 3950 60
-F35 "TEC_F0" O L 4800 4250 60
-F36 "ADC0_1" I L 4800 5950 60
-F37 "TEC_F1" O L 4800 4350 60
-F38 "DAC" O L 4800 5850 60
-F39 "TEC_F3" O L 4800 4550 60
-F40 "TEC_F2" O L 4800 4450 60
-F41 "LCD1" O L 4800 5250 60
-F42 "LCD2" O L 4800 5350 60
-F43 "LCD3" O L 4800 5450 60
-F44 "LCD_RS" O L 4800 5650 60
-F45 "LCD__EN" O L 4800 5750 60
-F46 "LCD4" O L 4800 5550 60
-F47 "LED2_R" O R 7050 6450 60
-F48 "LED2_G" O R 7050 6550 60
-F49 "LED2_B" O R 7050 6650 60
-F50 "LED3_R" O R 7050 6800 60
-F51 "LED3_G" O R 7050 6900 60
-F52 "LED3_B" O R 7050 7000 60
-F53 "GPIO4" B L 4800 1450 60
-F54 "CAN_RD" I L 4800 5100 60
-F55 "CAN_TD" O L 4800 5000 60
-F56 "GPIO5" B L 4800 1550 60
-F57 "WAKEUP0" I L 4800 2150 60
-F58 "TEC_COL1" O L 4800 4050 60
-F59 "TEC_COL2" O L 4800 4150 60
-F60 "GPIO6" B L 4800 1650 60
-F61 "ADC0_3" I L 4800 4800 60
-F62 "ISP" I R 7050 1700 60
-F63 "ADC0_2" I L 4800 4900 60
-F64 "GPIO8" B L 4800 1850 60
-F65 "GPIO7" B L 4800 1750 60
-F66 "USB_DEBUG_VBUS" O L 4800 6600 60
-F67 "I2C_SCL" O L 4800 3050 60
-F68 "I2C_SDA" B L 4800 2950 60
-F69 "LED1_R" O R 7050 6100 60
-F70 "LED1_G" O R 7050 6200 60
-F71 "LED1_B" O R 7050 6300 60
-F72 "LED0_R" O R 7050 5750 60
-F73 "LED0_G" O R 7050 5850 60
-F74 "LED0_B" O R 7050 5950 60
+F25 "RS485_RXD" I R 7050 3050 60
+F26 "RESET" O L 4800 6850 60
+F27 "PULS_0" I R 7050 5200 60
+F28 "PULS_1" I R 7050 5300 60
+F29 "PULS_2" I R 7050 5400 60
+F30 "PULS_3" I R 7050 5500 60
+F31 "TEC_COL0" O L 4800 3950 60
+F32 "TEC_F0" O L 4800 4250 60
+F33 "ADC0_1" I L 4800 5950 60
+F34 "TEC_F1" O L 4800 4350 60
+F35 "DAC" O L 4800 5850 60
+F36 "TEC_F3" O L 4800 4550 60
+F37 "TEC_F2" O L 4800 4450 60
+F38 "LCD1" O L 4800 5250 60
+F39 "LCD2" O L 4800 5350 60
+F40 "LCD3" O L 4800 5450 60
+F41 "LCD_RS" O L 4800 5650 60
+F42 "LCD__EN" O L 4800 5750 60
+F43 "LCD4" O L 4800 5550 60
+F44 "LED2_R" O R 7050 6450 60
+F45 "LED2_G" O R 7050 6550 60
+F46 "LED2_B" O R 7050 6650 60
+F47 "LED3_R" O R 7050 6800 60
+F48 "LED3_G" O R 7050 6900 60
+F49 "LED3_B" O R 7050 7000 60
+F50 "GPIO4" B L 4800 1450 60
+F51 "CAN_RD" I L 4800 5100 60
+F52 "CAN_TD" O L 4800 5000 60
+F53 "GPIO5" B L 4800 1550 60
+F54 "WAKEUP0" I L 4800 2150 60
+F55 "TEC_COL1" O L 4800 4050 60
+F56 "TEC_COL2" O L 4800 4150 60
+F57 "GPIO6" B L 4800 1650 60
+F58 "ADC0_3" I L 4800 4800 60
+F59 "ISP" I R 7050 1700 60
+F60 "ADC0_2" I L 4800 4900 60
+F61 "GPIO8" B L 4800 1850 60
+F62 "GPIO7" B L 4800 1750 60
+F63 "USB_DEBUG_VBUS" O L 4800 6600 60
+F64 "I2C_SCL" O L 4800 3050 60
+F65 "I2C_SDA" B L 4800 2950 60
+F66 "LED1_R" O R 7050 6100 60
+F67 "LED1_G" O R 7050 6200 60
+F68 "LED1_B" O R 7050 6300 60
+F69 "LED0_R" O R 7050 5750 60
+F70 "LED0_G" O R 7050 5850 60
+F71 "LED0_B" O R 7050 5950 60
+F72 "RS485_TXD" O R 7050 2950 60
 $EndSheet
 Wire Wire Line
@@
 Text Label 7450 3700 0    60   ~ 0
 USB_VBUS
+Wire Wire Line
+	7050 2950 8300 2950
 $EndSCHEMATC
