File: PCB/EDU-NXP/fuente.sch (KiCad schematic (older format))
At the start: 10 parts, among them U4 NCP1117ST33T3G

Commit message: Versión con algunas mejoras
Parts:
- added D13: PMEG3020EH, ~, symbol DIODESCH
- renumbered D45 to D12
Connections:
- net +5V: now also D13.2 (K)
- new net USB_VBUS3: D13.1 (A)
Changed lines of the file:
@@
 $Descr A4 11693 8268
 encoding utf-8
-Sheet 5 7
+Sheet 7 7
 Title "CIAA Fuente de alimentación"
-Date "10 jun 2014"
+Date "12 jun 2014"
 Rev "1.0"
 Comp ""
@@
 $EndComp
 $Comp
-L GND #PWR085
+L GND #PWR0118
 U 1 1 52B78C6E
 P 5200 4500
-F 0 "#PWR085" H 5200 4500 30  0001 C CNN
+F 0 "#PWR0118" H 5200 4500 30  0001 C CNN
 F 1 "GND" H 5200 4430 30  0001 C CNN
 F 2 "" H 5200 4500 60  0000 C CNN
@@
 $EndComp
 $Comp
-L GND #PWR086
+L GND #PWR0119
 U 1 1 52B78D01
 P 6050 4600
-F 0 "#PWR086" H 6050 4600 30  0001 C CNN
+F 0 "#PWR0119" H 6050 4600 30  0001 C CNN
 F 1 "GND" H 6050 4530 30  0001 C CNN
 F 2 "" H 6050 4600 60  0000 C CNN
@@
 $EndComp
 $Comp
-L GND #PWR087
+L GND #PWR0120
 U 1 1 52B78D23
 P 6650 4500
-F 0 "#PWR087" H 6650 4500 30  0001 C CNN
+F 0 "#PWR0120" H 6650 4500 30  0001 C CNN
 F 1 "GND" H 6650 4430 30  0001 C CNN
 F 2 "" H 6650 4500 60  0000 C CNN
@@
 $EndComp
 $Comp
-L GND #PWR088
+L GND #PWR0121
 U 1 1 52CF8853
 P 5500 5250
-F 0 "#PWR088" H 5500 5250 30  0001 C CNN
+F 0 "#PWR0121" H 5500 5250 30  0001 C CNN
 F 1 "GND" H 5500 5180 30  0001 C CNN
 F 2 "" H 5500 5250 60  0000 C CNN
@@
 Fuente de alimentación a través del puerto USB \nTensiones de salida: 5V y 3.3V\n
 Wire Wire Line
-	4100 3800 4100 4200
+	4100 3800 4100 4600
 Wire Wire Line
 	4900 4100 4900 4150
@@
 $EndComp
 $Comp
-L GND #PWR089
+L GND #PWR0122
 U 1 1 52D1F0B5
 P 4900 4700
-F 0 "#PWR089" H 4900 4700 30  0001 C CNN
+F 0 "#PWR0122" H 4900 4700 30  0001 C CNN
 F 1 "GND" H 4900 4630 30  0001 C CNN
 F 2 "" H 4900 4700 60  0000 C CNN
@@
 	7850 3700 7850 4100
 $Comp
-L +5V #PWR090
+L +5V #PWR0123
 U 1 1 52DEA2A1
 P 5200 3700
-F 0 "#PWR090" H 5200 3790 20  0001 C CNN
+F 0 "#PWR0123" H 5200 3790 20  0001 C CNN
 F 1 "+5V" H 5200 3790 30  0000 C CNN
 F 2 "" H 5200 3700 60  0000 C CNN
@@
 $EndComp
 $Comp
-L +3.3V #PWR091
+L +3.3V #PWR0124
 U 1 1 52DEA2B0
 P 6650 3700
-F 0 "#PWR091" H 6650 3660 30  0001 C CNN
+F 0 "#PWR0124" H 6650 3660 30  0001 C CNN
 F 1 "+3.3V" H 6650 3810 30  0000 C CNN
 F 2 "" H 6650 3700 60  0000 C CNN
@@
 $EndComp
 $Comp
-L +3.3VADC #PWR092
+L +3.3VADC #PWR0125
 U 1 1 52DEA2BF
 P 7850 3700
-F 0 "#PWR092" H 7850 3820 20  0001 C CNN
+F 0 "#PWR0125" H 7850 3820 20  0001 C CNN
 F 1 "+3.3VADC" H 7850 3790 30  0000 C CNN
 F 2 "" H 7850 3700 60  0000 C CNN
@@
 $EndComp
 $Comp
-L GND #PWR093
+L GND #PWR0126
 U 1 1 52DEAAB6
 P 7000 4750
-F 0 "#PWR093" H 7000 4750 30  0001 C CNN
+F 0 "#PWR0126" H 7000 4750 30  0001 C CNN
 F 1 "GND" H 7000 4680 30  0001 C CNN
 F 2 "" H 7000 4750 60  0000 C CNN
@@
 	7000 4600 7050 4600
 $Comp
-L GNDA #PWR094
+L GNDA #PWR0127
 U 1 1 52DEAAE6
 P 7850 4750
-F 0 "#PWR094" H 7850 4750 40  0001 C CNN
+F 0 "#PWR0127" H 7850 4750 40  0001 C CNN
 F 1 "GNDA" H 7850 4680 40  0000 C CNN
 F 2 "" H 7850 4750 60  0000 C CNN
@@
 	7850 4600 7750 4600
 $Comp
-L PWR_FLAG #FLG095
+L PWR_FLAG #FLG0128
 U 1 1 52DFF728
 P 5350 3700
-F 0 "#FLG095" H 5350 3795 30  0001 C CNN
+F 0 "#FLG0128" H 5350 3795 30  0001 C CNN
 F 1 "PWR_FLAG" H 5350 3880 30  0000 C CNN
 F 2 "" H 5350 3700 60  0000 C CNN
@@
 Connection ~ 5200 3750
 $Comp
-L PWR_FLAG #FLG096
+L PWR_FLAG #FLG0129
 U 1 1 52DFF757
 P 8100 3700
-F 0 "#FLG096" H 8100 3795 30  0001 C CNN
+F 0 "#FLG0129" H 8100 3795 30  0001 C CNN
 F 1 "PWR_FLAG" H 8100 3880 30  0000 C CNN
 F 2 "" H 8100 3700 60  0000 C CNN
@@
 Connection ~ 7850 3750
 $Comp
-L PWR_FLAG #FLG097
+L PWR_FLAG #FLG0130
 U 1 1 52DFF7BB
 P 7850 4550
-F 0 "#FLG097" H 7850 4645 30  0001 C CNN
+F 0 "#FLG0130" H 7850 4645 30  0001 C CNN
 F 1 "PWR_FLAG" H 7850 4730 30  0000 C CNN
 F 2 "" H 7850 4550 60  0000 C CNN
@@
 USB_VBUS2
 $Comp
-L DIODESCH D45
+L DIODESCH D12
 U 1 1 52EACD19
 P 3750 4200
-F 0 "D45" H 3750 4300 40  0000 C CNN
+F 0 "D12" H 3750 4300 40  0000 C CNN
 F 1 "PMEG3020EH" H 3750 4100 40  0000 C CNN
 F 2 "~" H 3750 4200 60  0000 C CNN
@@
 	4100 4200 3950 4200
 $Comp
-L PWR_FLAG #FLG098
+L PWR_FLAG #FLG0131
 U 1 1 52EACD22
 P 3500 4150
-F 0 "#FLG098" H 3500 4245 30  0001 C CNN
+F 0 "#FLG0131" H 3500 4245 30  0001 C CNN
 F 1 "PWR_FLAG" H 3500 4330 30  0000 C CNN
 F 2 "" H 3500 4150 60  0000 C CNN
@@
 	3950 3800 4100 3800
 $Comp
-L PWR_FLAG #FLG099
+L PWR_FLAG #FLG0132
 U 1 1 52EACD34
 P 3500 3750
-F 0 "#FLG099" H 3500 3845 30  0001 C CNN
+F 0 "#FLG0132" H 3500 3845 30  0001 C CNN
 F 1 "PWR_FLAG" H 3500 3930 30  0000 C CNN
 F 2 "" H 3500 3750 60  0000 C CNN
@@
 Connection ~ 4100 4200
 Connection ~ 4100 4100
+Text HLabel 3450 4600 0    60   Input ~ 0
+USB_VBUS3
+$Comp
+L DIODESCH D13
+U 1 1 539A74B5
+P 3750 4600
+F 0 "D13" H 3750 4700 40  0000 C CNN
+F 1 "PMEG3020EH" H 3750 4500 40  0000 C CNN
+F 2 "~" H 3750 4600 60  0000 C CNN
+F 3 "~" H 3750 4600 60  0000 C CNN
+	1    3750 4600
+	1    0    0    -1
+$EndComp
+Wire Wire Line
+	3450 4600 3550 4600
+Wire Wire Line
+	4100 4600 3950 4600
+$Comp
+L PWR_FLAG #FLG0133
+U 1 1 539A74BD
+P 3500 4550
+F 0 "#FLG0133" H 3500 4645 30  0001 C CNN
+F 1 "PWR_FLAG" H 3500 4730 30  0000 C CNN
+F 2 "" H 3500 4550 60  0000 C CNN
+F 3 "" H 3500 4550 60  0000 C CNN
+	1    3500 4550
+	1    0    0    -1
+$EndComp
+Wire Wire Line
+	3500 4550 3500 4600
+Connection ~ 3500 4600
 $EndSCHEMATC
