File: PCB/EDU-NXP/fuente.sch (KiCad schematic (older format))
At the start: 11 parts, among them U4 NCP1117ST33T3G

Commit message: Primera versión
Primera versión de la EDU - CIAA
Changed lines of the file:
@@
 $Descr A4 11693 8268
 encoding utf-8
-Sheet 7 7
-Title "CIAA Fuente de alimentación"
-Date "13 jun 2014"
+Sheet 5 7
+Title "EDU CIAA Fuente de alimentación"
+Date "14 jun 2014"
 Rev "1.0"
 Comp ""
@@
 $EndComp
 $Comp
-L GND #PWR081
+L GND #PWR027
 U 1 1 52B78C6E
 P 5200 4500
-F 0 "#PWR081" H 5200 4500 30  0001 C CNN
+F 0 "#PWR027" H 5200 4500 30  0001 C CNN
 F 1 "GND" H 5200 4430 30  0001 C CNN
 F 2 "" H 5200 4500 60  0000 C CNN
@@
 $EndComp
 $Comp
-L GND #PWR082
+L GND #PWR028
 U 1 1 52B78D01
 P 6050 4600
-F 0 "#PWR082" H 6050 4600 30  0001 C CNN
+F 0 "#PWR028" H 6050 4600 30  0001 C CNN
 F 1 "GND" H 6050 4530 30  0001 C CNN
 F 2 "" H 6050 4600 60  0000 C CNN
@@
 $EndComp
 $Comp
-L GND #PWR083
+L GND #PWR029
 U 1 1 52B78D23
 P 6650 4500
-F 0 "#PWR083" H 6650 4500 30  0001 C CNN
+F 0 "#PWR029" H 6650 4500 30  0001 C CNN
 F 1 "GND" H 6650 4430 30  0001 C CNN
 F 2 "" H 6650 4500 60  0000 C CNN
@@
 $EndComp
 $Comp
-L GND #PWR084
+L GND #PWR030
 U 1 1 52CF8853
 P 5500 5250
-F 0 "#PWR084" H 5500 5250 30  0001 C CNN
+F 0 "#PWR030" H 5500 5250 30  0001 C CNN
 F 1 "GND" H 5500 5180 30  0001 C CNN
 F 2 "" H 5500 5250 60  0000 C CNN
@@
 $EndComp
 $Comp
-L GND #PWR085
+L GND #PWR031
 U 1 1 52D1F0B5
 P 4900 4700
-F 0 "#PWR085" H 4900 4700 30  0001 C CNN
+F 0 "#PWR031" H 4900 4700 30  0001 C CNN
 F 1 "GND" H 4900 4630 30  0001 C CNN
 F 2 "" H 4900 4700 60  0000 C CNN
@@
 	7850 3700 7850 4100
 $Comp
-L +5V #PWR086
+L +5V #PWR032
 U 1 1 52DEA2A1
 P 5200 3700
-F 0 "#PWR086" H 5200 3790 20  0001 C CNN
+F 0 "#PWR032" H 5200 3790 20  0001 C CNN
 F 1 "+5V" H 5200 3790 30  0000 C CNN
 F 2 "" H 5200 3700 60  0000 C CNN
@@
 $EndComp
 $Comp
-L +3.3V #PWR087
+L +3.3V #PWR033
 U 1 1 52DEA2B0
 P 6650 3700
-F 0 "#PWR087" H 6650 3660 30  0001 C CNN
+F 0 "#PWR033" H 6650 3660 30  0001 C CNN
 F 1 "+3.3V" H 6650 3810 30  0000 C CNN
 F 2 "" H 6650 3700 60  0000 C CNN
@@
 $EndComp
 $Comp
-L +3.3VADC #PWR088
+L +3.3VADC #PWR034
 U 1 1 52DEA2BF
 P 7850 3700
-F 0 "#PWR088" H 7850 3820 20  0001 C CNN
+F 0 "#PWR034" H 7850 3820 20  0001 C CNN
 F 1 "+3.3VADC" H 7850 3790 30  0000 C CNN
 F 2 "" H 7850 3700 60  0000 C CNN
@@
 $EndComp
 $Comp
-L GND #PWR089
+L GND #PWR035
 U 1 1 52DEAAB6
 P 7000 4750
-F 0 "#PWR089" H 7000 4750 30  0001 C CNN
+F 0 "#PWR035" H 7000 4750 30  0001 C CNN
 F 1 "GND" H 7000 4680 30  0001 C CNN
 F 2 "" H 7000 4750 60  0000 C CNN
@@
 	7000 4600 7050 4600
 $Comp
-L GNDA #PWR090
+L GNDA #PWR036
 U 1 1 52DEAAE6
 P 7850 4750
-F 0 "#PWR090" H 7850 4750 40  0001 C CNN
+F 0 "#PWR036" H 7850 4750 40  0001 C CNN
 F 1 "GNDA" H 7850 4680 40  0000 C CNN
 F 2 "" H 7850 4750 60  0000 C CNN
@@
 	7850 4600 7750 4600
 $Comp
-L PWR_FLAG #FLG091
+L PWR_FLAG #FLG037
 U 1 1 52DFF728
 P 5350 3700
-F 0 "#FLG091" H 5350 3795 30  0001 C CNN
+F 0 "#FLG037" H 5350 3795 30  0001 C CNN
 F 1 "PWR_FLAG" H 5350 3880 30  0000 C CNN
 F 2 "" H 5350 3700 60  0000 C CNN
@@
 Connection ~ 5200 3750
 $Comp
-L PWR_FLAG #FLG092
+L PWR_FLAG #FLG038
 U 1 1 52DFF757
 P 8100 3700
-F 0 "#FLG092" H 8100 3795 30  0001 C CNN
+F 0 "#FLG038" H 8100 3795 30  0001 C CNN
 F 1 "PWR_FLAG" H 8100 3880 30  0000 C CNN
 F 2 "" H 8100 3700 60  0000 C CNN
@@
 Connection ~ 7850 3750
 $Comp
-L PWR_FLAG #FLG093
+L PWR_FLAG #FLG039
 U 1 1 52DFF7BB
 P 7850 4550
-F 0 "#FLG093" H 7850 4645 30  0001 C CNN
+F 0 "#FLG039" H 7850 4645 30  0001 C CNN
 F 1 "PWR_FLAG" H 7850 4730 30  0000 C CNN
 F 2 "" H 7850 4550 60  0000 C CNN
@@
 	4100 4200 3950 4200
 $Comp
-L PWR_FLAG #FLG094
+L PWR_FLAG #FLG040
 U 1 1 52EACD22
 P 3500 4150
-F 0 "#FLG094" H 3500 4245 30  0001 C CNN
+F 0 "#FLG040" H 3500 4245 30  0001 C CNN
 F 1 "PWR_FLAG" H 3500 4330 30  0000 C CNN
 F 2 "" H 3500 4150 60  0000 C CNN
@@
 	3950 3800 4100 3800
 $Comp
-L PWR_FLAG #FLG095
+L PWR_FLAG #FLG041
 U 1 1 52EACD34
 P 3500 3750
-F 0 "#FLG095" H 3500 3845 30  0001 C CNN
+F 0 "#FLG041" H 3500 3845 30  0001 C CNN
 F 1 "PWR_FLAG" H 3500 3930 30  0000 C CNN
 F 2 "" H 3500 3750 60  0000 C CNN
@@
 	4100 4600 3950 4600
 $Comp
-L PWR_FLAG #FLG096
+L PWR_FLAG #FLG042
 U 1 1 539A74BD
 P 3500 4550
-F 0 "#FLG096" H 3500 4645 30  0001 C CNN
+F 0 "#FLG042" H 3500 4645 30  0001 C CNN
 F 1 "PWR_FLAG" H 3500 4730 30  0000 C CNN
 F 2 "" H 3500 4550 60  0000 C CNN
@@
 	3500 4550 3500 4600
 Connection ~ 3500 4600
+$Comp
+L PWR_FLAG #FLG043
+U 1 1 539BAEDC
+P 7000 4600
+F 0 "#FLG043" H 7000 4695 30  0001 C CNN
+F 1 "PWR_FLAG" H 7000 4780 30  0000 C CNN
+F 2 "" H 7000 4600 60  0000 C CNN
+F 3 "" H 7000 4600 60  0000 C CNN
+	1    7000 4600
+	1    0    0    -1
+$EndComp
 $EndSCHEMATC

Commit message: Borrador del PCB
Parts:
- removed D13: PMEG3020EH, ~, symbol DIODESCH
- renumbered C17 to C5, C18 to C6, D5 to D4, D12 to D5, D4 to D6, FB6 to FB3, FB20 to FB4, R22 to R57, U4 to U3, ZA14 to ZA1
Changed lines of the file:
@@
 Sheet 5 7
 Title "EDU CIAA Fuente de alimentación"
-Date "14 jun 2014"
+Date "2 jul 2014"
 Rev "1.0"
 Comp ""
@@
 $EndDescr
 $Comp
-L NCP1117ST33T3G U4
+L NCP1117ST33T3G U3
 U 1 1 52B779B3
 P 6050 4150
-F 0 "U4" H 6200 3954 40  0000 C CNN
+F 0 "U3" H 6200 3954 40  0000 C CNN
 F 1 "NCP1117ST33T3G" H 6050 4350 40  0000 C CNN
 F 2 "~" H 6050 4150 60  0000 C CNN
@@
 $EndComp
 $Comp
-L CAPAPOL C17
+L CAPAPOL C5
 U 1 1 52B78C68
 P 5200 4300
-F 0 "C17" H 5250 4400 40  0000 L CNN
+F 0 "C5" H 5250 4400 40  0000 L CNN
 F 1 "330uF" H 5250 4200 40  0000 L CNN
 F 2 "~" H 5300 4150 30  0000 C CNN
@@
 $EndComp
 $Comp
-L GND #PWR027
+L GND #PWR022
 U 1 1 52B78C6E
 P 5200 4500
-F 0 "#PWR027" H 5200 4500 30  0001 C CNN
+F 0 "#PWR022" H 5200 4500 30  0001 C CNN
 F 1 "GND" H 5200 4430 30  0001 C CNN
 F 2 "" H 5200 4500 60  0000 C CNN
@@
 $EndComp
 $Comp
-L GND #PWR028
+L GND #PWR023
 U 1 1 52B78D01
 P 6050 4600
-F 0 "#PWR028" H 6050 4600 30  0001 C CNN
+F 0 "#PWR023" H 6050 4600 30  0001 C CNN
 F 1 "GND" H 6050 4530 30  0001 C CNN
 F 2 "" H 6050 4600 60  0000 C CNN
@@
 $EndComp
 $Comp
-L CAPAPOL C18
+L CAPAPOL C6
 U 1 1 52B78D18
 P 6650 4300
-F 0 "C18" H 6700 4400 40  0000 L CNN
+F 0 "C6" H 6700 4400 40  0000 L CNN
 F 1 "10uF" H 6700 4200 40  0000 L CNN
 F 2 "~" H 6750 4150 30  0000 C CNN
@@
 $EndComp
 $Comp
-L GND #PWR029
+L GND #PWR024
 U 1 1 52B78D23
 P 6650 4500
-F 0 "#PWR029" H 6650 4500 30  0001 C CNN
+F 0 "#PWR024" H 6650 4500 30  0001 C CNN
 F 1 "GND" H 6650 4430 30  0001 C CNN
 F 2 "" H 6650 4500 60  0000 C CNN
@@
 $EndComp
 $Comp
-L LED D4
+L LED D6
 U 1 1 52CF8844
 P 5500 4900
-F 0 "D4" H 5500 5000 50  0000 C CNN
+F 0 "D6" H 5500 5000 50  0000 C CNN
 F 1 "LED red" H 5500 4800 50  0000 C CNN
 F 2 "~" H 5500 4900 60  0000 C CNN
@@
 $EndComp
 $Comp
-L R R22
+L R R57
 U 1 1 52CF884A
 P 5500 4400
-F 0 "R22" V 5580 4400 40  0000 C CNN
+F 0 "R57" V 5580 4400 40  0000 C CNN
 F 1 "1k" V 5507 4401 40  0000 C CNN
 F 2 "~" V 5430 4400 30  0000 C CNN
@@
 $EndComp
 $Comp
-L GND #PWR030
+L GND #PWR025
 U 1 1 52CF8853
 P 5500 5250
-F 0 "#PWR030" H 5500 5250 30  0001 C CNN
+F 0 "#PWR025" H 5500 5250 30  0001 C CNN
 F 1 "GND" H 5500 5180 30  0001 C CNN
 F 2 "" H 5500 5250 60  0000 C CNN
@@
 Fuente de alimentación a través del puerto USB \nTensiones de salida: 5V y 3.3V\n
 Wire Wire Line
-	4100 3800 4100 4600
-Wire Wire Line
 	4900 4100 4900 4150
 Wire Wire Line
@@
 	6450 4100 7050 4100
 $Comp
-L TVS ZA14
+L TVS ZA1
 U 1 1 52D1F0AA
 P 4900 4400
-F 0 "ZA14" H 4900 4550 60  0000 C CNN
+F 0 "ZA1" H 4900 4550 60  0000 C CNN
 F 1 "SMAZ5V6" H 4900 4250 60  0000 C CNN
 F 2 "~" H 4900 4400 60  0000 C CNN
@@
 $EndComp
 $Comp
-L GND #PWR031
+L GND #PWR026
 U 1 1 52D1F0B5
 P 4900 4700
-F 0 "#PWR031" H 4900 4700 30  0001 C CNN
+F 0 "#PWR026" H 4900 4700 30  0001 C CNN
 F 1 "GND" H 4900 4630 30  0001 C CNN
 F 2 "" H 4900 4700 60  0000 C CNN
@@
 	4900 4700 4900 4650
 $Comp
-L FILTER FB6
+L FILTER FB3
 U 1 1 52D8A97B
 P 7400 4100
-F 0 "FB6" H 7400 4250 60  0000 C CNN
+F 0 "FB3" H 7400 4250 60  0000 C CNN
 F 1 "MMZ1608B601C" H 7400 4000 60  0000 C CNN
 F 2 "~" H 7400 4100 60  0000 C CNN
@@
 	7850 3700 7850 4100
 $Comp
-L +5V #PWR032
+L +5V #PWR027
 U 1 1 52DEA2A1
 P 5200 3700
-F 0 "#PWR032" H 5200 3790 20  0001 C CNN
+F 0 "#PWR027" H 5200 3790 20  0001 C CNN
 F 1 "+5V" H 5200 3790 30  0000 C CNN
 F 2 "" H 5200 3700 60  0000 C CNN
@@
 $EndComp
 $Comp
-L +3.3V #PWR033
+L +3.3V #PWR028
 U 1 1 52DEA2B0
 P 6650 3700
-F 0 "#PWR033" H 6650 3660 30  0001 C CNN
+F 0 "#PWR028" H 6650 3660 30  0001 C CNN
 F 1 "+3.3V" H 6650 3810 30  0000 C CNN
 F 2 "" H 6650 3700 60  0000 C CNN
@@
 $EndComp
 $Comp
-L +3.3VADC #PWR034
+L +3.3VADC #PWR029
 U 1 1 52DEA2BF
 P 7850 3700
-F 0 "#PWR034" H 7850 3820 20  0001 C CNN
+F 0 "#PWR029" H 7850 3820 20  0001 C CNN
 F 1 "+3.3VADC" H 7850 3790 30  0000 C CNN
 F 2 "" H 7850 3700 60  0000 C CNN
@@
 $EndComp
 $Comp
-L FILTER FB20
+L FILTER FB4
 U 1 1 52DEAAB0
 P 7400 4600
-F 0 "FB20" H 7400 4750 60  0000 C CNN
+F 0 "FB4" H 7400 4750 60  0000 C CNN
 F 1 "MMZ1608B601C" H 7400 4500 60  0000 C CNN
 F 2 "~" H 7400 4600 60  0000 C CNN
@@
 $EndComp
 $Comp
-L GND #PWR035
+L GND #PWR030
 U 1 1 52DEAAB6
 P 7000 4750
-F 0 "#PWR035" H 7000 4750 30  0001 C CNN
+F 0 "#PWR030" H 7000 4750 30  0001 C CNN
 F 1 "GND" H 7000 4680 30  0001 C CNN
 F 2 "" H 7000 4750 60  0000 C CNN
@@
 	7000 4600 7050 4600
 $Comp
-L GNDA #PWR036
+L GNDA #PWR031
 U 1 1 52DEAAE6
 P 7850 4750
-F 0 "#PWR036" H 7850 4750 40  0001 C CNN
+F 0 "#PWR031" H 7850 4750 40  0001 C CNN
 F 1 "GNDA" H 7850 4680 40  0000 C CNN
 F 2 "" H 7850 4750 60  0000 C CNN
@@
 	7850 4600 7750 4600
 $Comp
-L PWR_FLAG #FLG037
+L PWR_FLAG #FLG032
 U 1 1 52DFF728
 P 5350 3700
-F 0 "#FLG037" H 5350 3795 30  0001 C CNN
+F 0 "#FLG032" H 5350 3795 30  0001 C CNN
 F 1 "PWR_FLAG" H 5350 3880 30  0000 C CNN
 F 2 "" H 5350 3700 60  0000 C CNN
@@
 Connection ~ 5200 3750
 $Comp
-L PWR_FLAG #FLG038
+L PWR_FLAG #FLG033
 U 1 1 52DFF757
 P 8100 3700
-F 0 "#FLG038" H 8100 3795 30  0001 C CNN
+F 0 "#FLG033" H 8100 3795 30  0001 C CNN
 F 1 "PWR_FLAG" H 8100 3880 30  0000 C CNN
 F 2 "" H 8100 3700 60  0000 C CNN
@@
 Connection ~ 7850 3750
 $Comp
-L PWR_FLAG #FLG039
+L PWR_FLAG #FLG034
 U 1 1 52DFF7BB
 P 7850 4550
-F 0 "#FLG039" H 7850 4645 30  0001 C CNN
+F 0 "#FLG034" H 7850 4645 30  0001 C CNN
 F 1 "PWR_FLAG" H 7850 4730 30  0000 C CNN
 F 2 "" H 7850 4550 60  0000 C CNN
@@
 USB_VBUS2
 $Comp
-L DIODESCH D12
+L DIODESCH D5
 U 1 1 52EACD19
 P 3750 4200
-F 0 "D12" H 3750 4300 40  0000 C CNN
+F 0 "D5" H 3750 4300 40  0000 C CNN
 F 1 "PMEG3020EH" H 3750 4100 40  0000 C CNN
 F 2 "~" H 3750 4200 60  0000 C CNN
@@
 	4100 4200 3950 4200
 $Comp
-L PWR_FLAG #FLG040
+L PWR_FLAG #FLG035
 U 1 1 52EACD22
 P 3500 4150
-F 0 "#FLG040" H 3500 4245 30  0001 C CNN
+F 0 "#FLG035" H 3500 4245 30  0001 C CNN
 F 1 "PWR_FLAG" H 3500 4330 30  0000 C CNN
 F 2 "" H 3500 4150 60  0000 C CNN
@@
 USB_VBUS
 $Comp
-L DIODESCH D5
+L DIODESCH D4
 U 1 1 52EACD2B
 P 3750 3800
-F 0 "D5" H 3750 3900 40  0000 C CNN
+F 0 "D4" H 3750 3900 40  0000 C CNN
 F 1 "PMEG3020EH" H 3750 3700 40  0000 C CNN
 F 2 "~" H 3750 3800 60  0000 C CNN
@@
 	3950 3800 4100 3800
 $Comp
-L PWR_FLAG #FLG041
+L PWR_FLAG #FLG036
 U 1 1 52EACD34
 P 3500 3750
-F 0 "#FLG041" H 3500 3845 30  0001 C CNN
+F 0 "#FLG036" H 3500 3845 30  0001 C CNN
 F 1 "PWR_FLAG" H 3500 3930 30  0000 C CNN
 F 2 "" H 3500 3750 60  0000 C CNN
@@
 	3500 3750 3500 3800
 Connection ~ 3500 3800
-Connection ~ 4100 4200
 Connection ~ 4100 4100
-Text HLabel 3450 4600 0    60   Input ~ 0
-USB_VBUS3
-$Comp
-L DIODESCH D13
-U 1 1 539A74B5
-P 3750 4600
-F 0 "D13" H 3750 4700 40  0000 C CNN
-F 1 "PMEG3020EH" H 3750 4500 40  0000 C CNN
-F 2 "~" H 3750 4600 60  0000 C CNN
-F 3 "~" H 3750 4600 60  0000 C CNN
-	1    3750 4600
-	1    0    0    -1
-$EndComp
-Wire Wire Line
-	3450 4600 3550 4600
-Wire Wire Line
-	4100 4600 3950 4600
-$Comp
-L PWR_FLAG #FLG042
-U 1 1 539A74BD
-P 3500 4550
-F 0 "#FLG042" H 3500 4645 30  0001 C CNN
-F 1 "PWR_FLAG" H 3500 4730 30  0000 C CNN
-F 2 "" H 3500 4550 60  0000 C CNN
-F 3 "" H 3500 4550 60  0000 C CNN
-	1    3500 4550
-	1    0    0    -1
-$EndComp
-Wire Wire Line
-	3500 4550 3500 4600
-Connection ~ 3500 4600
-$Comp
-L PWR_FLAG #FLG043
+$Comp
+L PWR_FLAG #FLG037
 U 1 1 539BAEDC
 P 7000 4600
-F 0 "#FLG043" H 7000 4695 30  0001 C CNN
+F 0 "#FLG037" H 7000 4695 30  0001 C CNN
 F 1 "PWR_FLAG" H 7000 4780 30  0000 C CNN
 F 2 "" H 7000 4600 60  0000 C CNN
@@
 	1    0    0    -1
 $EndComp
+Wire Wire Line
+	4100 3800 4100 4200
 $EndSCHEMATC
