File: PCB/EDU-NXP/gpio.sch (KiCad schematic (older format))
At the start: 10 parts, among them P1 CONN_20X2, P2 CONN_20X2

Commit message: Versión con algunas mejoras
Connections:
- net SPI_SCK: now reaches P2.25
Changed lines of the file:
@@
 Sheet 6 7
 Title "CIAA GPIO/SPI/I2C/USB/ANALOG"
-Date "10 jun 2014"
+Date "12 jun 2014"
 Rev "1.0"
 Comp ""
@@
 $EndComp
 $Comp
-L +3.3V #PWR080
+L +3.3V #PWR0113
 U 1 1 52CA1E6C
 P 3250 2600
-F 0 "#PWR080" H 3250 2560 30  0001 C CNN
+F 0 "#PWR0113" H 3250 2560 30  0001 C CNN
 F 1 "+3.3V" H 3250 2710 30  0000 C CNN
 F 2 "" H 3250 2600 60  0000 C CNN
@@
 	3550 3950 3550 5200
 $Comp
-L +5V #PWR081
+L +5V #PWR0114
 U 1 1 52CA305A
 P 10450 2450
-F 0 "#PWR081" H 10450 2540 20  0001 C CNN
+F 0 "#PWR0114" H 10450 2540 20  0001 C CNN
 F 1 "+5V" H 10450 2540 30  0000 C CNN
 F 2 "" H 10450 2450 60  0000 C CNN
@@
 Conectores de expansión LVTTL.\nEn formato de pines, 2.54mm de pitch.
 $Comp
-L GNDA #PWR082
+L GNDA #PWR0115
 U 1 1 52DEB0D0
 P 3550 5200
-F 0 "#PWR082" H 3550 5200 40  0001 C CNN
+F 0 "#PWR0115" H 3550 5200 40  0001 C CNN
 F 1 "GNDA" H 3550 5130 40  0000 C CNN
 F 2 "" H 3550 5200 60  0000 C CNN
@@
 $EndComp
 $Comp
-L +3.3V #PWR083
+L +3.3V #PWR0116
 U 1 1 539535E0
 P 8100 2450
-F 0 "#PWR083" H 8100 2410 30  0001 C CNN
+F 0 "#PWR0116" H 8100 2410 30  0001 C CNN
 F 1 "+3.3V" H 8100 2560 30  0000 C CNN
 F 2 "" H 8100 2450 60  0000 C CNN
@@
 	5500 2600 5450 2600
 $Comp
-L +5V #PWR084
+L +5V #PWR0117
 U 1 1 539535EE
 P 5500 2600
-F 0 "#PWR084" H 5500 2690 20  0001 C CNN
+F 0 "#PWR0117" H 5500 2690 20  0001 C CNN
 F 1 "+5V" H 5500 2690 30  0000 C CNN
 F 2 "" H 5500 2600 60  0000 C CNN
@@
 	3550 3950 4000 3950
 Connection ~ 3550 4150
+Text HLabel 8100 4100 0    60   Input ~ 0
+SPI_SCK
+Wire Wire Line
+	8100 4100 8950 4100
 $EndSCHEMATC
