File: PCB/EDU-NXP/gpio.sch (KiCad schematic (older format))
At the start: 10 parts, among them P1 CONN_20X2, P2 CONN_20X2

Commit message: Primera versión
Primera versión de la EDU - CIAA
Parts:
- removed TH9: MF-MSMF110-2, ~, symbol THERMISTOR
- added GS1, GS10, GS11, GS12, GS13, GS14, GS15, GS16, GS17, GS18, GS19, GS2, GS20, GS21, GS22, GS23, GS24, GS25, GS26, GS27, GS28, GS29, GS3, GS30, GS31, GS32, GS33, GS34, GS35, GS36, GS37, GS38, GS39, GS40, GS41, GS42, GS43, GS44, GS45, GS6, GS7, GS8, GS9: GS2, symbol GS2
- added R1, R105, R106, R107, R108, R109, R110, R111, R112, R2, R3, R4, R5, R56, R57, R58, R59, R6, R60, R61, R62, R63, R64, R65, R66, R67, R68, R69, R7, R70, R71, R72, R73, R74, R75, R76, R77, R78, R79, R80, R81, R82, R83: R, ~, symbol R
- added TH3: MF-MSMF110-2, ~, symbol THERMISTOR
Connections:
- net +3.3V: now also TH2.2, TH8.2; no longer TH2.1, TH8.1
- net +5V: now also TH3.2
- net CAN_RD: now also GS42.2 (G2), R109.1; no longer P2.4 (P4)
- net CAN_TD: now also GS43.2 (G2), R110.1; no longer P2.6 (P6)
- net ENET_CRS_DV: now also GS34.1 (G1), R80.2; no longer P2.9 (P9)
- net ENET_MDIO: now also GS35.1 (G1), R81.2; no longer P2.11 (P11)
- net ENET_REF_CLK: now also GS25.1 (G1), R71.2; no longer P2.15 (P15)
- net ENET_RXD0: now also GS33.1 (G1), R79.2; no longer P2.7 (P7)
- net ENET_RXD1: now also GS31.1 (G1), R77.2; no longer P2.3 (P3)
- net ENET_TXD0: now also GS36.1 (G1), R82.2; no longer P2.13 (P13)
- net ENET_TXD1: now also GS26.1 (G1), R72.2; no longer P2.17 (P17)
- net ENET_TX_EN: now also GS32.1 (G1), R78.2; no longer P2.5 (P5)
- net GNDA: now also P1.23 (P23)
- net GPIO0: now also GS37.2 (G2), R83.1; no longer P1.4 (P4)
- net GPIO1: now also GS38.2 (G2), R105.1; no longer P1.6 (P6)
- net GPIO2: now also GS39.2 (G2), R106.1; no longer P1.8 (P8)
- net GPIO3: now also GS40.2 (G2), R107.1; no longer P1.10 (P10)
- net GPIO4: now also GS41.2 (G2), R108.1; no longer P1.12 (P12)
- net GPIO5: now also GS45.2 (G2), R112.1; no longer P2.12 (P12)
- net GPIO6: now also GS19.2 (G2), R65.1; no longer P2.14 (P14)
- net GPIO7: now also GS20.2 (G2), R66.1; no longer P2.16 (P16)
- net GPIO8: now also GS21.2 (G2), R67.1; no longer P2.18 (P18)
- net I2C_SCL: now also GS1.1 (G1), R1.2; no longer P1.3 (P3)
- net I2C_SDA: now also GS2.1 (G1), R2.2; no longer P1.5 (P5)
- net ISP: now also GS12.1 (G1), R58.2; no longer P1.23 (P23)
- net LCD1: now also GS13.2 (G2), R59.1; no longer P1.14 (P14)
- net LCD2: now also GS14.2 (G2), R60.1; no longer P1.16 (P16)
- net LCD3: now also GS15.2 (G2), R61.1; no longer P1.18 (P18)
- net LCD4: now also GS16.2 (G2), R62.1; no longer P1.20 (P20)
- net LCD_EN: now also GS18.2 (G2), R64.1; no longer P1.24 (P24)
- net LCD_RS: now also GS17.2 (G2), R63.1; no longer P1.22 (P22)
- net RS232_RXD: now also GS23.2 (G2), R69.1; no longer P2.28 (P28)
- net RS232_TXD: now also GS22.2 (G2), R68.1; no longer P2.26 (P26)
- net SPI_MISO: now also GS28.1 (G1), R74.2; no longer P2.21 (P21)
- net SPI_MOSI: now also GS29.1 (G1), R75.2; no longer P2.23 (P23)
- net SPI_SCK: now also GS30.1 (G1), R76.2; no longer P2.25
- net TEC_COL0: now also GS3.1 (G1), R3.2; no longer P1.7 (P7)
- net TEC_COL1: now also GS6.1 (G1), R4.2; no longer P1.9 (P9)
- net TEC_COL2: now also GS7.1 (G1), R5.2; no longer P1.11 (P11)
- net TEC_F0: now also GS8.1 (G1), R6.2; no longer P1.13 (P13)
- net TEC_F1: now also GS9.1 (G1), R7.2; no longer P1.15 (P15)
- net TEC_F2: now also GS10.1 (G1), R56.2; no longer P1.17 (P17)
- net TEC_F3: now also GS11.1 (G1), R57.2; no longer P1.19 (P19)
- net WAKEUP: now also GS44.2 (G2), R111.1; no longer P2.8 (P8)
- net at P1.1 (P1): now also TH8.1; no longer TH8.2
- net at P2.2 (P2): now also TH3.1
- net at P2.1 (P1): now also TH2.1; no longer TH2.2
- net at P1.21 (P21): now also GS12.2 (G2), R58.1
- net GND: now reaches P1.26 (P26)
- net GND: now also P1.28 (P28), P1.30 (P30), P1.32 (P32), P1.34 (P34), P1.36 (P36), P1.38 (P38), P1.40 (P40), P2.24 (P24), P2.26 (P26), P2.27 (P27), P2.28 (P28), P2.29 (P29), P2.30 (P30), P2.31 (P31), P2.32 (P32), P2.33 (P33), P2.34 (P34), P2.35 (P35), P2.36 (P36), P2.37 (P37), P2.38 (P38), P2.39 (P39), P2.40 (P40)
- net at P2.10 (P10): now also GS45.1 (G1), R112.2
- net at P2.19 (P19): now also GS27.2 (G2), R73.1
- net at P2.20 (P20): now also GS23.1 (G1), R69.2
- net at P2.22 (P22): now also GS24.1 (G1), R70.2
- new net: GS40.1 (G1), P1.10 (P10), R107.2
- new net: GS7.2 (G2), P1.11 (P11), R5.1
- new net: GS41.1 (G1), P1.12 (P12), R108.2
- new net: GS8.2 (G2), P1.13 (P13), R6.1
- new net: GS13.1 (G1), P1.14 (P14), R59.2
- new net: GS9.2 (G2), P1.15 (P15), R7.1
- new net: GS14.1 (G1), P1.16 (P16), R60.2
- new net: GS10.2 (G2), P1.17 (P17), R56.1
- new net: GS15.1 (G1), P1.18 (P18), R61.2
- new net: GS11.2 (G2), P1.19 (P19), R57.1
- new net: GS16.1 (G1), P1.20 (P20), R62.2
- new net: GS17.1 (G1), P1.22 (P22), R63.2
- new net: GS18.1 (G1), P1.24 (P24), R64.2
- new net: GS1.2 (G2), P1.3 (P3), R1.1
- new net: GS37.1 (G1), P1.4 (P4), R83.2
- new net: GS2.2 (G2), P1.5 (P5), R2.1
- new net: GS38.1 (G1), P1.6 (P6), R105.2
- new net: GS3.2 (G2), P1.7 (P7), R3.1
- new net: GS39.1 (G1), P1.8 (P8), R106.2
- new net: GS6.2 (G2), P1.9 (P9), R4.1
- new net: GS35.2 (G2), P2.11 (P11), R81.1
- new net: GS19.1 (G1), P2.12 (P12), R65.2
- new net: GS36.2 (G2), P2.13 (P13), R82.1
- new net: GS20.1 (G1), P2.14 (P14), R66.2
- new net: GS25.2 (G2), P2.15 (P15), R71.1
- new net: GS21.1 (G1), P2.16 (P16), R67.2
- new net: GS26.2 (G2), P2.17 (P17), R72.1
- new net: GS22.1 (G1), P2.18 (P18), R68.2
- new net: GS28.2 (G2), P2.21 (P21), R74.1
- new net: GS29.2 (G2), P2.23 (P23), R75.1
- new net: GS30.2 (G2), P2.25, R76.1
- new net: GS31.2 (G2), P2.3 (P3), R77.1
- new net: GS42.1 (G1), P2.4 (P4), R109.2
- new net: GS32.2 (G2), P2.5 (P5), R78.1
- new net: GS43.1 (G1), P2.6 (P6), R110.2
- new net: GS33.2 (G2), P2.7 (P7), R79.1
- new net: GS44.1 (G1), P2.8 (P8), R111.2
- new net: GS34.2 (G2), P2.9 (P9), R80.1
- new net ENET_MDC: GS27.1 (G1), R73.2
- new net RESET: GS24.2 (G2), R70.1
Other:
- note added: "La distribución de los pines, se modificará al momento de rutear el PCB\n"
- moved on the sheet: P1, P2, R12, R13, R14, R15, TH1, TH8

Commit message: Borrador del PCB
Parts:
- renumbered GS12 to GS10, GS37 to GS11, GS38 to GS12, GS39 to GS13, GS40 to GS14, GS41 to GS15, GS13 to GS16, GS14 to GS17, GS15 to GS18, GS16 to GS19, GS17 to GS20, GS18 to GS21, GS31 to GS22, GS32 to GS23, GS33 to GS24, GS34 to GS25, GS35 to GS26, GS36 to GS27, GS25 to GS28, GS26 to GS29, GS27 to GS30, GS28 to GS31, GS29 to GS32, GS30 to GS33, GS42 to GS34, GS43 to GS35, GS44 to GS36, GS45 to GS37, GS19 to GS38, GS20 to GS39, GS6 to GS4, GS21 to GS40, GS22 to GS41, GS23 to GS42, GS24 to GS43, GS7 to GS5, GS8 to GS6, GS9 to GS7, GS10 to GS8, GS11 to GS9, R1 to R10, R2 to R11, R3 to R12, R4 to R13, R5 to R14, R6 to R15, R7 to R16, R56 to R17, R57 to R18, R58 to R19, R12 to R20, R13 to R21, R14 to R22, R15 to R23, R83 to R24, R105 to R25, R106 to R26, R107 to R27, R108 to R28, R59 to R29, R60 to R30, R61 to R31, R62 to R32, R63 to R33, R64 to R34, R77 to R35, R78 to R36, R79 to R37, R80 to R38, R81 to R39, R82 to R40, R71 to R41, R72 to R42, R73 to R43, R74 to R44, R75 to R45, R76 to R46, R109 to R47, R110 to R48, R111 to R49, R112 to R50, R65 to R51, R66 to R52, R67 to R53, R68 to R54, R69 to R55, R70 to R56, TH8 to TH1, TH1 to TH2, TH2 to TH3, TH3 to TH4
