File: PCB/EDU-NXP/rsS485_rs232_can.sch (KiCad schematic (older format))
At the start: 22 parts, among them J2 TB_1X3, U5 MAX3072

Commit message: Borrador del PCB
Parts:
- renumbered C21 to C1, C22 to C2, D8 to D1, D6 to D2, D7 to D3, J2 to J1, JP3 to JP1, JP1 to JP2, JP2 to JP3, R34 to R1, R36 to R2, R37 to R3, R33 to R4, R38 to R5, R32 to R6, R35 to R7, R39 to R8, R40 to R9, U5 to U1
Changed lines of the file:
@@
 Sheet 2 7
 Title "EDU CIAA RS485"
-Date "14 jun 2014"
+Date "2 jul 2014"
 Rev "1.0"
 Comp ""
@@
 $EndDescr
 $Comp
-L MAX3072 U5
+L MAX3072 U1
 U 1 1 52C5B349
 P 5200 3800
-F 0 "U5" H 5000 4050 30  0000 C CNN
+F 0 "U1" H 5000 4050 30  0000 C CNN
 F 1 "MAX3072" H 5400 3550 30  0000 C CNN
 F 2 "SOIC8" H 5200 3800 35  0001 C CIN
@@
 $EndComp
 $Comp
-L C_MINI C22
+L C_MINI C2
 U 1 1 52C5B34A
 P 4850 3350
-F 0 "C22" V 4850 3450 30  0000 C CNN
+F 0 "C2" V 4850 3450 30  0000 C CNN
 F 1 "100nF" V 4900 3500 30  0000 C CNN
 F 2 "~" H 4850 3350 60  0000 C CNN
@@
 $EndComp
 $Comp
-L R_MINI R33
+L R_MINI R4
 U 1 1 52C5B34C
 P 5850 3200
-F 0 "R33" V 5900 3100 30  0000 C CNN
+F 0 "R4" V 5900 3100 30  0000 C CNN
 F 1 "100K" V 5850 3100 30  0000 C CNN
 F 2 "~" H 5850 3200 60  0000 C CNN
@@
 $EndComp
 $Comp
-L R_MINI R35
+L R_MINI R7
 U 1 1 52C5B34D
 P 6100 3900
-F 0 "R35" V 6100 3800 30  0000 C CNN
+F 0 "R7" V 6100 3800 30  0000 C CNN
 F 1 "120" V 6050 3800 30  0000 C CNN
 F 2 "~" H 6100 3900 60  0000 C CNN
@@
 $EndComp
 $Comp
-L R_MINI R38
+L R_MINI R5
 U 1 1 52C5B34E
 P 5850 4350
-F 0 "R38" V 5850 4250 30  0000 C CNN
+F 0 "R5" V 5850 4250 30  0000 C CNN
 F 1 "100K" V 5800 4250 30  0000 C CNN
 F 2 "~" H 5850 4350 60  0000 C CNN
@@
 $EndComp
 $Comp
-L ESD D8
+L ESD D1
 U 1 1 52C5B34F
 P 6400 3150
-F 0 "D8" V 6400 3050 30  0000 C CNN
+F 0 "D1" V 6400 3050 30  0000 C CNN
 F 1 "PSD12C" V 6350 3000 30  0000 C CNN
 F 2 "~" H 6400 3150 60  0000 C CNN
@@
 $EndComp
 $Comp
-L ESD D6
+L ESD D2
 U 1 1 52C5B350
 P 6400 3750
-F 0 "D6" V 6400 3650 30  0000 C CNN
+F 0 "D2" V 6400 3650 30  0000 C CNN
 F 1 "PSD12C" V 6350 3600 30  0000 C CNN
 F 2 "~" H 6400 3750 60  0000 C CNN
@@
 $EndComp
 $Comp
-L ESD D7
+L ESD D3
 U 1 1 52C5B351
 P 6400 4350
-F 0 "D7" V 6400 4250 30  0000 C CNN
+F 0 "D3" V 6400 4250 30  0000 C CNN
 F 1 "PSD12C" V 6350 4200 30  0000 C CNN
 F 2 "~" H 6400 4350 60  0000 C CNN
@@
 $EndComp
 $Comp
-L R_MINI R32
+L R_MINI R6
 U 1 1 52C5B362
 P 6100 3100
-F 0 "R32" V 6150 3000 30  0000 C CNN
+F 0 "R6" V 6150 3000 30  0000 C CNN
 F 1 "680" V 6100 3000 30  0000 C CNN
 F 2 "~" H 6100 3100 60  0000 C CNN
@@
 $EndComp
 $Comp
-L R_MINI R39
+L R_MINI R8
 U 1 1 52C5B363
 P 6100 4450
-F 0 "R39" V 6100 4350 30  0000 C CNN
+F 0 "R8" V 6100 4350 30  0000 C CNN
 F 1 "680" V 6050 4350 30  0000 C CNN
 F 2 "~" H 6100 4450 60  0000 C CNN
@@
 $EndComp
 $Comp
-L JUMPER-2 JP2
+L JUMPER-2 JP3
 U 1 1 52C5B366
 P 6100 3650
-F 0 "JP2" V 6100 3575 30  0000 C CNN
+F 0 "JP3" V 6100 3575 30  0000 C CNN
 F 1 "JUMPER-2" H 6100 3650 30  0001 C CNN
 F 2 "~" H 6100 3650 60  0000 C CNN
@@
 $EndComp
 $Comp
-L JUMPER-2 JP1
+L JUMPER-2 JP2
 U 1 1 52C5B367
 P 6100 3350
-F 0 "JP1" V 6100 3275 30  0000 C CNN
+F 0 "JP2" V 6100 3275 30  0000 C CNN
 F 1 "JUMPER-2" H 6100 3350 30  0001 C CNN
 F 2 "~" H 6100 3350 60  0000 C CNN
@@
 RS485
 $Comp
-L TB_1X3 J2
+L TB_1X3 J1
 U 1 1 52C5B37D
 P 7850 3750
-F 0 "J2" H 7950 4050 60  0000 C CNN
+F 0 "J1" H 7950 4050 60  0000 C CNN
 F 1 "TB_1X3" H 7900 3250 60  0000 C CNN
 F 2 "" H 7800 3800 60  0000 C CNN
@@
 JP1, JP2, JP4: cortocircuitar en\ncaso que sea el último nodo de la red.
 $Comp
-L R_MINI R37
+L R_MINI R3
 U 1 1 52C5B37E
 P 4600 4300
-F 0 "R37" V 4600 4200 30  0000 C CNN
+F 0 "R3" V 4600 4200 30  0000 C CNN
 F 1 "4K7" V 4550 4200 30  0000 C CNN
 F 2 "~" H 4600 4300 60  0000 C CNN
@@
 $EndComp
 $Comp
-L R_MINI R36
+L R_MINI R2
 U 1 1 52C5B380
 P 4300 4300
-F 0 "R36" V 4300 4200 30  0000 C CNN
+F 0 "R2" V 4300 4200 30  0000 C CNN
 F 1 "4K7" V 4250 4200 30  0000 C CNN
 F 2 "~" H 4300 4300 60  0000 C CNN
@@
 $EndComp
 $Comp
-L JUMPER-2 JP3
+L JUMPER-2 JP1
 U 1 1 52C5B382
 P 4450 4000
-F 0 "JP3" H 4450 3925 30  0000 C CNN
+F 0 "JP1" H 4450 3925 30  0000 C CNN
 F 1 "JUMPER-2" H 4450 4000 30  0001 C CNN
 F 2 "~" H 4450 4000 60  0000 C CNN
@@
 $EndComp
 $Comp
-L CP_MINI C21
+L CP_MINI C1
 U 1 1 52C5B383
 P 4650 3350
-F 0 "C21" V 4650 3500 30  0000 C CNN
+F 0 "C1" V 4650 3500 30  0000 C CNN
 F 1 "10uF / 6V3" V 4700 3550 25  0000 C CNN
 F 2 "~" H 4650 3350 60  0000 C CNN
@@
 $EndComp
 $Comp
-L R_MINI R40
+L R_MINI R9
 U 1 1 52C5B387
 P 7450 4350
-F 0 "R40" H 7450 4200 30  0000 C CNN
+F 0 "R9" H 7450 4200 30  0000 C CNN
 F 1 "100 / 1/2W" H 7450 4250 30  0000 C CNN
 F 2 "~" H 7450 4350 60  0000 C CNN
@@
 Connection ~ 5200 4600
 $Comp
-L R_MINI R34
+L R_MINI R1
 U 1 1 52C5B38C
 P 4150 3500
-F 0 "R34" V 4150 3400 30  0000 C CNN
+F 0 "R1" V 4150 3400 30  0000 C CNN
 F 1 "4K7" V 4100 3400 30  0000 C CNN
 F 2 "~" H 4150 3500 60  0000 C CNN
@@
 	0    -1   -1   0
 $EndComp
-Wire Wire Line
-	4150 3600 4150 4100
-Connection ~ 4150 4100
 Wire Wire Line
 	4150 3350 4150 3400
@@
 	1    0    0    -1
 $EndComp
+Wire Wire Line
+	4150 3600 4150 3650
+Connection ~ 4150 3650
 $EndSCHEMATC
